File: SMDProtoBreakoutPanel.kicad_pcb (KiCad board)
At the start: 2 copper layers, 0 parts

Commit message: auto-backup 2026-07-28 01:26:33
Parts:
- added D1: SOD-123, Diode_SMD:D_SOD-123, F.Cu at (56.0, 65.0)
- added D2: SOD-123, Diode_SMD:D_SOD-123, F.Cu at (69.0, 65.0)
- added D3: SOD-323, Diode_SMD:D_SOD-323_HandSoldering, F.Cu at (56.0, 85.0)
- added D4: SOD-323, Diode_SMD:D_SOD-323_HandSoldering, F.Cu at (69.0, 85.0)
- added J1: 1x16, Connector_PinHeader_2.54mm:PinHeader_1x16_P2.54mm_Vertical, F.Cu at (2.54, 9.00)
- added J10: 1x02, Connector_PinHeader_2.54mm:PinHeader_1x02_P2.54mm_Vertical, F.Cu at (31.0, 71.5)
- added J11: 1x02, Connector_PinHeader_2.54mm:PinHeader_1x02_P2.54mm_Vertical, F.Cu at (44.0, 71.5)
- added J12: 1x02, Connector_PinHeader_2.54mm:PinHeader_1x02_P2.54mm_Vertical, F.Cu at (31.0, 79.0)
- added J13: 1x02, Connector_PinHeader_2.54mm:PinHeader_1x02_P2.54mm_Vertical, F.Cu at (44.0, 79.0)
- added J14: 1x02, Connector_PinHeader_2.54mm:PinHeader_1x02_P2.54mm_Vertical, F.Cu at (56.0, 71.5)
- added J15: 1x02, Connector_PinHeader_2.54mm:PinHeader_1x02_P2.54mm_Vertical, F.Cu at (69.0, 71.5)
- added J16: 1x02, Connector_PinHeader_2.54mm:PinHeader_1x02_P2.54mm_Vertical, F.Cu at (56.0, 79.0)
- added J17: 1x02, Connector_PinHeader_2.54mm:PinHeader_1x02_P2.54mm_Vertical, F.Cu at (69.0, 79.0)
- added J18: 1x08, Connector_PinHeader_2.54mm:PinHeader_1x08_P2.54mm_Vertical, F.Cu at (81.1, 66.1)
- added J19: 1x08, Connector_PinHeader_2.54mm:PinHeader_1x08_P2.54mm_Vertical, F.Cu at (93.9, 66.1)
- added J2: 1x16, Connector_PinHeader_2.54mm:PinHeader_1x16_P2.54mm_Vertical, F.Cu at (22.5, 6.00)
- added J3: 1x04, Connector_PinHeader_2.54mm:PinHeader_1x04_P2.54mm_Vertical, F.Cu at (31.0, 21.2)
- added J4: 1x04, Connector_PinHeader_2.54mm:PinHeader_1x04_P2.54mm_Vertical, F.Cu at (44.0, 21.2)
- added J5: 1x03, Connector_PinHeader_2.54mm:PinHeader_1x03_P2.54mm_Vertical, F.Cu at (56.5, 22.5)
- added J6: 1x03, Connector_PinHeader_2.54mm:PinHeader_1x03_P2.54mm_Vertical, F.Cu at (68.5, 22.5)
- added J7: 1x04, Connector_PinHeader_2.54mm:PinHeader_1x04_P2.54mm_Vertical, F.Cu at (94.5, 21.2)
- added J8: 1x03, Connector_PinHeader_2.54mm:PinHeader_1x03_P2.54mm_Vertical, F.Cu at (7.00, 72.5)
- added J9: 1x03, Connector_PinHeader_2.54mm:PinHeader_1x03_P2.54mm_Vertical, F.Cu at (18.0, 72.5)
- added MH1: MountingHole_3.2mm, MountingHole:MountingHole_3.2mm, F.Cu at (5.00, 5.00)
- added MH2: MountingHole_3.2mm, MountingHole:MountingHole_3.2mm, F.Cu at (95.0, 5.00)
- added MH3: MountingHole_3.2mm, MountingHole:MountingHole_3.2mm, F.Cu at (95.0, 95.0)
- added MH4: MountingHole_3.2mm, MountingHole:MountingHole_3.2mm, F.Cu at (5.00, 95.0)
- added R1: 0805, Resistor_SMD:R_0805_2012Metric_Pad1.20x1.40mm_HandSolder, F.Cu at (31.0, 65.0)
- added R2: 0805, Resistor_SMD:R_0805_2012Metric_Pad1.20x1.40mm_HandSolder, F.Cu at (44.0, 65.0)
- added R3: 0603, Resistor_SMD:R_0603_1608Metric_Pad0.98x0.95mm_HandSolder, F.Cu at (31.0, 85.0)
- added R4: 0603, Resistor_SMD:R_0603_1608Metric_Pad0.98x0.95mm_HandSolder, F.Cu at (44.0, 85.0)
- added U1: TQFP-32, Package_QFP:TQFP-32_7x7mm_P0.8mm, F.Cu at (12.5, 25.0)
- added U2: SOIC-8, Package_SO:SOIC-8_3.9x4.9mm_P1.27mm, F.Cu at (37.5, 25.0)
- added U3: SOT-23-6, Package_TO_SOT_SMD:SOT-23-6_Handsoldering, F.Cu at (62.5, 25.0)
- added U4: SOT-223, Package_TO_SOT_SMD:SOT-223-3_TabPin2, F.Cu at (87.5, 25.0)
- added U5: SC-70-6, Package_TO_SOT_SMD:SOT-363_SC-70-6, F.Cu at (12.5, 75.0)
- added U6: SOIC-16, Package_SO:SOIC-16_3.9x9.9mm_P1.27mm, F.Cu at (87.5, 75.0)
Routing:
- net S8_9: track 0.00 -> 13.9 mm
- net S8_16: track 0.00 -> 13.9 mm
- net S8_15: track 0.00 -> 10.3 mm
- net S8_10: track 0.00 -> 10.3 mm
- net S2_8: track 0.00 -> 6.99 mm
- net S2_5: track 0.00 -> 6.99 mm
- net S8_14: track 0.00 -> 6.91 mm
- net S8_11: track 0.00 -> 6.91 mm
- net S7_D2_1: track 0.00 -> 6.71 mm
- net S7_D1_1: track 0.00 -> 6.71 mm
- net S6_R2_1: track 0.00 -> 6.58 mm
- net S6_R1_1: track 0.00 -> 6.58 mm
- net S7_D4_1: track 0.00 -> 6.13 mm
- net S7_D3_1: track 0.00 -> 6.13 mm
- net S6_R4_1: track 0.00 -> 6.07 mm
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Other:
- board outline added: 100 x 100 mm
- copper layers 2 -> 4
- board text added: "0805 / 0603 Passive Breakout"
- board text added: "Diodes SOD-123 / SOD-323"
- board text added: "SC-70 to DIP-6"
- board text added: "SOIC-16 to DIP-16"
- board text added: "SOIC-8 to DIP-8"
- board text added: "SOT-223 to DIP-4"
- board text added: "SOT-23-6 to DIP-6"
- board text added: "TQFP-32 to DIP-32"
- board text added: "V-CUT"

Commit message: auto-backup 2026-07-28 02:26:40
Routing:
- net S1_17: track 0.00 -> 63.7 mm
- net S1_19: track 0.00 -> 58.4 mm
- net S1_32: track 0.00 -> 28.5 mm, vias 0 -> 1
- net S1_16: track 0.00 -> 23.2 mm
- net S1_30: track 0.00 -> 22.8 mm, vias 0 -> 1
- net S1_15: track 0.00 -> 20.4 mm
- net S8_15: track 10.3 -> 28.1 mm
- net S1_28: track 0.00 -> 17.1 mm, vias 0 -> 1
- net S1_20: track 0.00 -> 17.0 mm, vias 0 -> 1
- net S4_2: track 0.00 -> 16.0 mm, vias 0 -> 1
- net S1_1: track 0.00 -> 15.5 mm
- net S4_3: track 0.00 -> 14.8 mm, vias 0 -> 1
- net S4_1: track 0.00 -> 14.6 mm, vias 0 -> 1
- net S1_2: track 0.00 -> 14.4 mm
- net S8_11: track 6.91 -> 19.0 mm, vias 0 -> 2
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
Commit message: auto-backup 2026-07-28 03:26:36
Routing:
- net S1_14: track 0.00 -> 40.3 mm, vias 0 -> 1
- net S1_29: track 0.00 -> 25.3 mm, vias 0 -> 1
- net S1_31: track 0.00 -> 23.9 mm, vias 0 -> 1
- net S1_18: track 0.00 -> 19.3 mm, vias 0 -> 1
- net S8_10: track 0.00 -> 19.1 mm, vias 0 -> 1
- net S1_13: track 0.00 -> 14.6 mm, vias 0 -> 1
- net S1_27: track 0.00 -> 13.7 mm, vias 0 -> 1
- net S1_12: track 0.00 -> 12.3 mm, vias 0 -> 1
- net S1_3: track 0.00 -> 11.3 mm, vias 0 -> 1
- net S1_26: track 0.00 -> 11.3 mm, vias 0 -> 1
- net S1_11: track 0.00 -> 10.2 mm, vias 0 -> 1
- net S1_4: track 0.00 -> 9.86 mm, vias 0 -> 1
- net S6_R1_2: track 0.00 -> 9.76 mm
- net S1_10: track 0.00 -> 9.60 mm
- net S5_4: track 0.00 -> 8.07 mm, vias 0 -> 1
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
Commit message: auto-backup 2026-07-28 04:26:37
Routing:
- net S1_27: track 13.7 -> 66.5 mm
- net S1_26: track 11.3 -> 59.9 mm
- net S1_24: track 6.01 -> 50.6 mm, vias 1 -> 2
- net S1_23: track 6.06 -> 45.6 mm, vias 1 -> 2
- net S1_31: track 23.9 -> 57.6 mm
- net S1_18: track 19.3 -> 0.00 mm
- net S8_10: track 19.1 -> 33.3 mm
Changed lines of the file:
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@@
 	(segment
 		(start 89.975 78.175)
-		(end 92.8 80)
+		(end 91.5 78.175)
 		(width 0.4)
 		(layer "B.Cu")
@@
 	)
 	(segment
-		(start 95.5 80)
-		(end 95.5 68.65)
+		(start 96 86)
+		(end 96 68.65)
 		(width 0.4)
 		(layer "B.Cu")
@@
 	)
 	(segment
-		(start 92.8 80)
-		(end 95.5 80)
+		(start 91.5 86)
+		(end 96 86)
 		(width 0.4)
 		(layer "B.Cu")
@@
 	)
 	(segment
-		(start 95.5 68.65)
+		(start 96 68.65)
 		(end 93.86 68.65)
+		(width 0.4)
+		(layer "B.Cu")
+		(net "S8_10")
+	)
+	(segment
+		(start 91.5 78.175)
+		(end 91.5 86)
 		(width 0.4)
 		(layer "B.Cu")
@@
 	)
 	(segment
-		(start 16.6625 27)
-		(end 22.46 8.54)
-		(width 0.4)
-		(layer "B.Cu")
-		(net "S1_18")
-	)
-	(segment
 		(start 23.8161 12.4361)
 		(end 22.46 11.08)
@@
 		(net "S1_22")
 	)
+	(segment
+		(start 17.5 23)
+		(end 20 15)
+		(width 0.4)
+		(layer "F.Cu")
+		(net "S1_23")
+	)
+	(segment
+		(start 16.6625 23)
+		(end 17.5 23)
+		(width 0.4)
+		(layer "F.Cu")
+		(net "S1_23")
+	)
+	(via
+		(at 20 15)
+		(size 0.5)
+		(drill 0.3)
+		(layers "F.Cu" "B.Cu")
+		(net "S1_23")
+	)
 	(via
 		(at 16.6625 23)
@@
 	)
 	(segment
-		(start 16.6625 23)
+		(start 24.7 21.24)
 		(end 22.46 21.24)
 		(width 0.4)
@@
 		(net "S1_23")
 	)
+	(segment
+		(start 20 15)
+		(end 20 3.4)
+		(width 0.4)
+		(layer "B.Cu")
+		(net "S1_23")
+	)
+	(segment
+		(start 24.7 3.4)
+		(end 24.7 21.24)
+		(width 0.4)
+		(layer "B.Cu")
+		(net "S1_23")
+	)
+	(segment
+		(start 20 3.4)
+		(end 24.7 3.4)
+		(width 0.4)
+		(layer "B.Cu")
+		(net "S1_23")
+	)
+	(segment
+		(start 18 21.5)
+		(end 19 16)
+		(width 0.4)
+		(layer "F.Cu")
+		(net "S1_24")
+	)
+	(segment
+		(start 16.6625 22.2)
+		(end 18 21.5)
+		(width 0.4)
+		(layer "F.Cu")
+		(net "S1_24")
+	)
 	(via
 		(at 16.6625 22.2)
@@
 		(net "S1_24")
 	)
-	(segment
-		(start 16.6625 22.2)
+	(via
+		(at 19 16)
+		(size 0.5)
+		(drill 0.3)
+		(layers "F.Cu" "B.Cu")
+		(net "S1_24")
+	)
+	(segment
+		(start 19 16)
+		(end 19 2.8)
+		(width 0.4)
+		(layer "B.Cu")
+		(net "S1_24")
+	)
+	(segment
+		(start 25.4 23.78)
 		(end 22.46 23.78)
+		(width 0.4)
+		(layer "B.Cu")
+		(net "S1_24")
+	)
+	(segment
+		(start 19 2.8)
+		(end 25.4 2.8)
+		(width 0.4)
+		(layer "B.Cu")
+		(net "S1_24")
+	)
+	(segment
+		(start 25.4 2.8)
+		(end 25.4 23.78)
 		(width 0.4)
 		(layer "B.Cu")
@@
 	)
 	(via
-		(at 14.5 20.8375)
+		(at 14.5 20.2)
 		(size 0.5)
 		(drill 0.3)
@@
 	)
 	(segment
-		(start 14.5 20.8375)
+		(start 26.1 2.2)
+		(end 26.1 28.86)
+		(width 0.4)
+		(layer "B.Cu")
+		(net "S1_26")
+	)
+	(segment
+		(start 14.5 20.2)
+		(end 14.5 2.2)
+		(width 0.4)
+		(layer "B.Cu")
+		(net "S1_26")
+	)
+	(segment
+		(start 14.5 2.2)
+		(end 26.1 2.2)
+		(width 0.4)
+		(layer "B.Cu")
+		(net "S1_26")
+	)
+	(segment
+		(start 26.1 28.86)
 		(end 22.46 28.86)
 		(width 0.4)
@@
 	)
 	(segment
+		(start 26.8 1.6)
+		(end 26.8 31.4)
+		(width 0.4)
+		(layer "B.Cu")
+		(net "S1_27")
+	)
+	(segment
+		(start 13.7 1.6)
+		(end 26.8 1.6)
+		(width 0.4)
+		(layer "B.Cu")
+		(net "S1_27")
+	)
+	(segment
+		(start 26.8 31.4)
+		(end 22.46 31.4)
+		(width 0.4)
+		(layer "B.Cu")
+		(net "S1_27")
+	)
+	(segment
 		(start 13.7 20.8375)
-		(end 22.46 31.4)
+		(end 13.7 1.6)
 		(width 0.4)
 		(layer "B.Cu")
@@
 		(net "S1_30")
 	)
-	(via
-		(at 10.5 20.8375)
-		(size 0.5)
-		(drill 0.3)
-		(layers "F.Cu" "B.Cu")
+	(segment
+		(start 10.5 20.8375)
+		(end 10.5 26)
+		(width 0.4)
+		(layer "F.Cu")
 		(net "S1_31")
 	)
-	(segment
-		(start 10.5 20.8375)
+	(via
+		(at 10.5 26)
+		(size 0.5)
+		(drill 0.3)
+		(layers "F.Cu" "B.Cu")
+		(net "S1_31")
+	)
+	(segment
+		(start 24 49)
+		(end 24 41.56)
+		(width 0.4)
+		(layer "B.Cu")
+		(net "S1_31")
+	)
+	(segment
+		(start 7 49)
+		(end 24 49)
+		(width 0.4)
+		(layer "B.Cu")
+		(net "S1_31")
+	)
+	(segment
+		(start 7 26)
+		(end 7 49)
+		(width 0.4)
+		(layer "B.Cu")
+		(net "S1_31")
+	)
+	(segment
+		(start 10.5 26)
+		(end 7 26)
+		(width 0.4)
+		(layer "B.Cu")
+		(net "S1_31")
+	)
+	(segment
+		(start 24 41.56)
 		(end 22.46 41.56)
 		(width 0.4)
